File: KiCAD Files/buck_converter.kicad_sch (KiCad schematic)
At the start: 28 parts, among them U3 LM76003RNPR, U4 LM76003RNPR

Commit message: Ethernet routing pending
Parts:
- removed C31, C32: 68u, Footprints:RR71C680MDN1, symbol RR71C680MDN1:RR71C680MDN1KX
- added C7, C8: 68u, Footprints:10SVPC68MV, symbol 10SVPC68MV:10SVPC68MV
- added D1, D2: LED, Footprints:RC0805FR-07680RL, symbol Device:LED
- added R26, R27: 680, Footprints:RC0805FR-07680RL, symbol RC0805FR-07680RL:RC0805FR-07680RL
Connections:
- net +5V_Radxa: now also C7.1 (+), R26.2
- net +5V_WiFi: now also C8.1 (+), R27.2
- net GND: now also C7.2 (-), C8.2 (-), D1.1 (K), D2.1 (K)
- new net: D1.2 (A), R26.1
- new net: D2.2 (A), R27.1
