File: KiCAD Files/VTX.kicad_pcb (KiCad board)
At the start: 2 copper layers, 32 x 65 mm, 33 parts, among them J2 XT90PW-M, U1 LM76003RNPR, U2 LM76003RNPR

Commit message: USB Controller Ready
Routing:
- net GND: vias 16 -> 18
Changed lines of the file:
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@@
 		(layer "F.SilkS")
+	)
+	(gr_rect
+		(start 42 113)
+		(end 74 145)
+		(stroke
+			(width 0.1)
+			(type solid)
+		)
+		(fill no)
+		(layer "F.Adhes")
 	)
 	(gr_line
@@
 	)
 	(via
+		(at 64.603057 91.550001)
+		(size 0.6)
+		(drill 0.3)
+		(layers "F.Cu" "B.Cu")
+		(net "GND")
+	)
+	(via
 		(at 69.823557 94.110002)
 		(size 0.6)
@@
 	)
 	(via
-		(at 61.103057 90.590002)
+		(at 60.65 90.6072)
 		(size 0.6)
 		(drill 0.3)
@@
 		(size 0.6)
 		(drill 0.3)
+		(layers "F.Cu" "B.Cu")
+		(net "GND")
+	)
+	(via
+		(at 50.508056 104.710003)
+		(size 0.6)
+		(drill 0.3)

Commit message: Ethernet routing pending
Parts:
- removed the H1 at (69.5, 84.5)
- removed the H1 at (45.5, 84.5)
- removed the H1 at (45.5, 115.0)
- removed L1, L2: 6060_78439346150, Footprints:L78439346150
- added C17: 1uF, Footprints:CC0805KKX7R6BB225, F.Cu at (244.2, 114.0)
- added C18: 1uF, Footprints:CC0805KKX7R6BB225, F.Cu at (246.6, 117.0)
- added C19: 4.7u, Footprints:CS3225X7R475K101NRK, F.Cu at (257.8, 73.0)
- added C20: 4.7u, Footprints:CS3225X7R475K101NRK, F.Cu at (247.5, 87.8)
- added C21: 470n, Footprints:C0805X474K101T, F.Cu at (256.4, 69.3)
- added C22: 470n, Footprints:C0805X474K101T, F.Cu at (247.1, 84.3)
- added C23: 1u, Footprints:CC0603KRX5R6BB105, F.Cu at (266.8, 68.8)
- added C24: 1u, Footprints:CC0603KRX5R6BB105, F.Cu at (255.7, 85.3)
- added C25: 2.2uF, Footprints:CC0805KKX7R6BB225, F.Cu at (266.8, 70.4)
- added C26: 2.2uF, Footprints:CC0805KKX7R6BB225, F.Cu at (255.7, 87.1)
- added C27: 2.2uF, Footprints:CS1005X7R474K6R3NR, F.Cu at (266.2, 71.8)
- added C28: 2.2uF, Footprints:CS1005X7R474K6R3NR, F.Cu at (255.1, 88.5)
- added C29: 10p, Footprints:10pF16V, F.Cu at (262.0, 65.2)
- added C30: 10p, Footprints:10pF16V, F.Cu at (254.1, 81.8)
- added C33: 470n, Footprints:CL10A474KB8NNNC, F.Cu at (268.4, 76.6)
- added C34: 470n, Footprints:CL10A474KB8NNNC, F.Cu at (266.2, 89.5)
- added C35: 0.1u, Footprints:100nF0603, F.Cu at (245.9, 104.4)
- added C36: 1uF, Footprints:C0805X474K101T, F.Cu at (250.3, 117.4)
- added C37: 0.1u, Footprints:100nF0603, F.Cu at (256.3, 105.1)
- added C38: 0.1u, Footprints:100nF0603, F.Cu at (260.6, 107.5)
- added C39: 0.1u, Footprints:100nF0603, F.Cu at (250.0, 139.0)
- added C40: 0.1u, Footprints:100nF0603, F.Cu at (248.4, 144.3)
- added C41: 0.1u, Footprints:100nF0603, F.Cu at (248.4, 146.7)
- added D1: LED, Footprints:RC0805FR-07680RL, F.Cu at (273.0, 76.8)
- added D2: LED, Footprints:RC0805FR-07680RL, F.Cu at (270.9, 90.1)
- added FL1: BLM18PG121SN1D, Footprints:BLM18PG121SN1D, F.Cu at (257.0, 117.1)
- added FL2: BLM18PG121SN1D, Footprints:BLM18PG121SN1D, F.Cu at (260.8, 105.2)
- added FL3: BLM18PG121SN1D, Footprints:BLM18PG121SN1D, F.Cu at (251.0, 103.9)
- added H1: MountingHole, MountingHole:MountingHole_3mm, F.Cu at (243.8, 64.0)
- added H3: MountingHole, MountingHole:MountingHole_3mm, F.Cu at (276.7, 126.9)
- added H4: MountingHole, MountingHole:MountingHole_3mm, F.Cu at (243.7, 126.9)
- added IC1: LAN9500AI-ABZJ-TR, Footprints:LAN9500AI-ABZJ-TR, F.Cu at (250.8, 110.5)
- added IC2: LDK120C33R, Footprints:LDK120C33R, F.Cu at (244.1, 117.4)
- added J1: Conn_02x20_Odd_Even, Connector_PinHeader_2.54mm:PinHeader_2x20_P2.54mm_Vertical, F.Cu at (275.5, 71.4)
- added J3: Ethernet, Connector_JST:JST_GH_SM04B-GHS-TB_1x04-1MP_P1.25mm_Horizontal, F.Cu at (253.4, 128.1)
- added J4: Port3, Connector_JST:JST_GH_SM04B-GHS-TB_1x04-1MP_P1.25mm_Horizontal, F.Cu at (243.9, 93.2)
- added J5: Port4, Connector_JST:JST_GH_SM04B-GHS-TB_1x04-1MP_P1.25mm_Horizontal, F.Cu at (269.2, 127.9)
- added J6: UART, Connector_JST:JST_GH_SM06B-GHS-TB_1x06-1MP_P1.25mm_Horizontal, F.Cu at (253.2, 63.1)
- added J7: FAN, Connector_JST:JST_GH_SM02B-GHS-TB_1x02-1MP_P1.25mm_Horizontal, F.Cu at (267.6, 63.1)
- added L3: 6060_78439346150, Footprints:L78439346150, F.Cu at (264.0, 77.6)
- added L4: 6060_78439346150, Footprints:L78439346150, F.Cu at (261.1, 87.3)
- added R10: 105K, Footprints:RC1206FR-07105KL, F.Cu at (249.0, 81.9)
- added R11: 100K, Footprints:RC0402FR-07100KL, F.Cu at (265.6, 66.8)
- added R12: 100K, Footprints:RC0402FR-07100KL, F.Cu at (256.3, 83.5)
- added R13: 24K9, Footprints:AC0402FR-0724K9L, F.Cu at (263.6, 65.8)
- added R14: 24K9, Footprints:AC0402FR-0724K9L, F.Cu at (255.9, 81.8)
- added R15: 100K, Footprints:RC0402FR-07100KL, F.Cu at (260.2, 64.8)
- added R16: 100K, Footprints:RC0402FR-07100KL, F.Cu at (252.1, 82.4)
- added R17: 10K, Footprints:RC0603JR-0710KL, F.Cu at (244.1, 110.1)
- added R18: 10K, Footprints:RC0603JR-0710KL, F.Cu at (248.6, 104.6)
- added R19: 10K, Footprints:RC0603JR-0710KL, F.Cu at (255.3, 117.1)
- added R20: 49R9, Footprints:RC0805FR-0749R9L, F.Cu at (263.7, 109.4)
- added R21: 49R9, Footprints:RC0805FR-0749R9L, F.Cu at (265.8, 109.4)
- added R22: 49R9, Footprints:RC0805FR-0749R9L, F.Cu at (261.5, 139.4)
- added R23: 49R9, Footprints:RC0805FR-0749R9L, F.Cu at (258.6, 139.6)
- added R24: 75, Footprints:RC0805FR-0775RL, F.Cu at (272.3, 109.5)
- added R25: 75, Footprints:RC0805FR-0775RL, F.Cu at (270.2, 109.5)
- added R26: 680, Footprints:RC0805FR-07680RL, F.Cu at (270.8, 76.8)
- added R27: 680, Footprints:RC0805FR-07680RL, F.Cu at (268.5, 90.1)
- added R9: 105K, Footprints:RC1206FR-07105KL, F.Cu at (258.8, 68.2)
- added T1: H1102NL, Footprints:H1102NL, F.Cu at (268.0, 117.8)
- added U3: LM76003RNPR, Footprints:LM76003RNPR, F.Cu at (262.6, 70.5)
- added U4: LM76003RNPR, Footprints:LM76003RNPR, F.Cu at (251.5, 87.0)
- added Y1: ABMM2-12.000MHZ-E2-T, Footprints:ABMM2-12MHz, F.Cu at (272.6, 96.9)
- added Y2: 25MHz, Footprints:ABM7-25MHz, F.Cu at (255.2, 101.3)
- C1, C10: value 470n -> 0.1u; footprint Footprints:C0805X474K101T -> Footprints:100nF0603
- C11: value 1u -> 0.1u; footprint Footprints:CC0603KRX5R6BB105 -> Footprints:100nF0603
- C12: value 2.2uF -> 0.1u; footprint Footprints:CC0805KKX7R6BB225 -> Footprints:100nF0603
- C13: value 2.2uF -> 0.1u; footprint Footprints:CS1005X7R474K6R3NR -> Footprints:100nF0603
- C14: value 10p -> 0.1u; footprint Footprints:10pF16V -> Footprints:100nF0603
- C15: value 68u -> 0.1u; footprint Footprints:RR71C680MDN1 -> Footprints:100nF0603
- C16: value 470n -> 0.1u; footprint Footprints:CL10A474KB8NNNC -> Footprints:100nF0603
- C2: value 2.2uF -> 10u; footprint Footprints:CC0805KKX7R6BB225 -> Footprints:CL10A106KQ8NNNC
- C3: value 2.2uF -> 10u; footprint Footprints:CS1005X7R474K6R3NR -> Footprints:CL10A106KQ8NNNC
- C4: value 4.7u -> 33p; footprint Footprints:CS3225X7R475K101NRK -> Footprints:TCC0402COG330J500AT
- C5: value 470n -> 33p; footprint Footprints:CL10A474KB8NNNC -> Footprints:TCC0402COG330J500AT
- C6: value 10p -> 1n; footprint Footprints:10pF16V -> Footprints:C1206C102JGRACTU
- C7: value 1u -> 68u; footprint Footprints:CC0603KRX5R6BB105 -> Footprints:10SVPC68MV
- C8: footprint Footprints:RR71C680MDN1 -> Footprints:10SVPC68MV
- C9: value 4.7u -> 0.1u; footprint Footprints:CS3225X7R475K101NRK -> Footprints:100nF0603
- J2: value XT90PW-M -> XT30PW-M; footprint Footprints:AMASS_XT90PW-M -> Footprints:AMASS_XT30PW-M
- R1: value 105K -> 10K; footprint Footprints:RC1206FR-07105KL -> Footprints:RC0603JR-0710KL
- R2: value 24K9 -> 100K; footprint Footprints:AC0402FR-0724K9L -> Footprints:RC0402FR-07100KL
- R3: value 100K -> 2K7; footprint Footprints:RC0402FR-07100KL -> Footprints:RC0805FR-072K7L
- R5: value 105K -> 12K; footprint Footprints:RC1206FR-07105KL -> Footprints:RC0805FR-0712KL
- R6: value 100K -> 12K; footprint Footprints:RC0402FR-07100KL -> Footprints:RC0805FR-0712KL
- R7: value 24K9 -> 10K; footprint Footprints:AC0402FR-0724K9L -> Footprints:RC0603JR-0710KL
- R8: value 100K -> 10K; footprint Footprints:RC0402FR-07100KL -> Footprints:RC0603JR-0710KL
- U1: value LM76003RNPR -> BL-M8812EU2; footprint Footprints:LM76003RNPR -> Footprints:BL-M8812EU2
- U2: value LM76003RNPR -> FE1.1S-BQFN24B; footprint Footprints:LM76003RNPR -> Footprints:FE1.1S-BQFN24B
- moved C8 220.4 mm to (269.8, 85.6), turned to 0 degrees
- moved U2 216.7 mm to (267.0, 96.6)
- moved C7 214.7 mm to (271.2, 70.2), turned to -90 degrees
- moved R5 213.7 mm to (260.0, 110.7)
- moved C10 213.3 mm to (259.5, 109.0)
- moved H2 213.3 mm to (276.6, 63.8)
- moved C9 211.2 mm to (257.6, 107.5), turned to 0 degrees
- moved R6 208.8 mm to (258.8, 105.0), turned to 90 degrees
- moved C3 208.6 mm to (268.9, 101.8), turned to 0 degrees
- moved C6 206.3 mm to (267.9, 108.8), turned to -90 degrees
- moved C2 206.2 mm to (266.6, 100.9), turned to 90 degrees
- moved C12 206.0 mm to (259.7, 114.0), turned to 0 degrees
- moved C11 203.3 mm to (259.8, 112.5), turned to 0 degrees
- moved R1 200.2 mm to (268.9, 100.2)
- moved C13 200.0 mm to (253.7, 117.0)
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Connections:
- C1 pad 2: Input -> +5V_Radxa
- C10 pad 1: GND -> /USB Hub/ferrite
- C10 pad 2: Input -> GND
- C11 pad 1: GND -> /USB Hub/ferrite
- C11 pad 2: Net-(U2-BIAS) -> GND
- C12 pad 1: GND -> /USB Hub/ferrite
- C12 pad 2: Net-(U2-VCC) -> GND
- C13 pad 1: Net-(U2-CBOOT) -> +3V3
- C13 pad 2: Net-(C13-Pad2) -> GND
- C14 pad 1: Net-(U2-BIAS) -> +3V3
- C14 pad 2: Net-(U2-FB) -> GND
- C15 pad 1: Net-(U2-BIAS) -> +3V3
- C16 pad 1: Net-(U2-BIAS) -> +3V3
- C2 pad 2: Net-(U1-VCC) -> +5V_Radxa
- C3 pad 1: Net-(U1-CBOOT) -> /USB Hub/VD33F
- C3 pad 2: Net-(C3-Pad2) -> GND
- C4 pad 2: Input -> /USB Hub/XO
- C5 pad 1: Net-(U1-BIAS) -> GND
- C5 pad 2: GND -> /USB Hub/XI
- C6 pad 1: Net-(U1-BIAS) -> GND
- C6 pad 2: Net-(U1-FB) -> Net-(C6-Pad2)
- C7 pad 1: GND -> +5V_Radxa
- C7 pad 2: Net-(U1-BIAS) -> GND
- C8 pad 1: Net-(U1-BIAS) -> +5V_WiFi
- C9 pad 1: GND -> /USB Hub/ferrite
- C9 pad 2: Input -> GND
- R1 pad 1: Net-(U1-BIAS) -> /USB Hub/VD33F
- R1 pad 2: Net-(U1-PGOOD) -> Net-(U2-OVCJ)
- R2 pad 1: Net-(U1-FB) -> /USB Hub/VD33F
- R2 pad 2: GND -> Net-(U2-XRSTJ)
- R3 pad 1: Net-(U1-BIAS) -> GND
- R3 pad 2: Net-(U1-FB) -> Net-(U2-REXT)
- R4 pad 1: GND -> Net-(U2-BUSJ)
- R4 pad 2: Net-(U1-RT) -> /USB Hub/VD33F
- R5 pad 1: Net-(U2-BIAS) -> GND
- R5 pad 2: Net-(U2-PGOOD) -> Net-(IC1-EXRES)
- R6 pad 1: GND -> Net-(IC1-USBRBIAS)
- R6 pad 2: Net-(U2-RT) -> GND
- R7 pad 1: Net-(U2-FB) -> Net-(IC1-EECLK/PWR_SEL)
- R7 pad 2: GND -> +3V3
- R8 pad 1: Net-(U2-BIAS) -> Net-(IC1-EECS)
- R8 pad 2: Net-(U2-FB) -> GND
- U1 pad 1: Net-(C3-Pad2) -> GND
- U1 pad 2: Net-(C3-Pad2) -> /USB Hub/USB_WiFi_P
- U1 pad 3: Net-(C3-Pad2) -> /USB Hub/USB_WiFi_N
- U1 pad 4: Net-(C3-Pad2) -> GND
- U1 pad 5: Net-(C3-Pad2) -> unconnected-(U1-RESET-Pad5)
- U1 pad 6: Net-(U1-CBOOT) -> +5V_WiFi
- U1 pad 7: unconnected-(U1-NC-Pad7) -> +5V_WiFi
- U1 pad 8: Net-(U1-VCC) -> GND
- U2 pad 1: Net-(C13-Pad2) -> Net-(U2-OVCJ)
- U2 pad 10: Net-(U2-RT) -> /USB Hub/USB_WiFi_P
- U2 pad 11: unconnected-(U2-SS_TRK-Pad11) -> /USB Hub/USB1_N
- U2 pad 12: Net-(U2-FB) -> /USB Hub/USB1_P
- U2 pad 13: GND -> Net-(U2-REXT)
- U2 pad 14: GND -> /USBD_UP_N
- U2 pad 15: GND -> /USBD_UP_P
- U2 pad 16: Net-(U2-PGOOD) -> Net-(U2-XRSTJ)
- U2 pad 17: GND -> +5V_Radxa
- U2 pad 18: Input -> Net-(U2-BUSJ)
- U2 pad 19: unconnected-(U2-NC-Pad19) -> +5V_Radxa
- U2 pad 2: Net-(C13-Pad2) -> unconnected-(U2-TESTJ-Pad2)
- U2 pad 20: Input -> /USB Hub/VD33F
- U2 pad 21: Input -> unconnected-(U2-DRV-Pad21)
- U2 pad 22: Input -> unconnected-(U2-LED1-Pad22)
- U2 pad 24: GND -> unconnected-(U2-PWRJ-Pad24)
- U2 pad 3: Net-(C13-Pad2) -> /USB Hub/XOUT
- U2 pad 4: Net-(C13-Pad2) -> /USB Hub/XIN
- U2 pad 5: Net-(C13-Pad2) -> /USB Hub/USB4_N
- U2 pad 6: Net-(U2-CBOOT) -> /USB Hub/USB4_P
- U2 pad 7: unconnected-(U2-NC-Pad7) -> /USB Hub/USB3_N
- U2 pad 8: Net-(U2-VCC) -> /USB Hub/USB3_P
- U2 pad 9: Net-(U2-BIAS) -> /USB Hub/USB_WiFi_N
Routing:
- net +5V_Radxa: track 0.00 -> 149.5 mm, vias 0 -> 2
- net /UART4_RX: track 0.00 -> 51.2 mm, vias 0 -> 4
- net +3V3: track 0.00 -> 49.0 mm, vias 0 -> 5
- net /UART4_TX: track 0.00 -> 46.4 mm, vias 0 -> 2
- net Input: track 83.4 -> 39.1 mm
- net +5V_WiFi: track 0.00 -> 39.4 mm, vias 0 -> 17
- net /USB Hub/USB1_N: track 0.00 -> 34.1 mm, vias 0 -> 2
- net /USB Hub/USB4_P: track 0.00 -> 32.8 mm, vias 0 -> 2
- net /USB Hub/VDDCORE: track 0.00 -> 32.7 mm, vias 0 -> 3
- net /USB Hub/USB4_N: track 0.00 -> 32.7 mm, vias 0 -> 2
- net /USB Hub/USB1_P: track 0.00 -> 32.3 mm, vias 0 -> 2
- net Net-(U1-BIAS): track 31.4 -> 0.00 mm
- net /USB Hub/TX_P: track 0.00 -> 30.3 mm
- net /USB Hub/ferrite: track 0.00 -> 30.0 mm, vias 0 -> 5
- net /USB Hub/TX_N: track 0.00 -> 29.5 mm
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- added copper zone on F.Cu, net +5V_Radxa
- removed copper zone on B.Cu, net GND
Other:
- board size 32 x 65 mm -> 40 x 70 mm
- board text removed: "C10"
- board text removed: "R2"

Commit message: Final Push
Parts:
- removed C40, C41: 0.1u, Footprints:100nF0603
- moved C39 36.9 mm to (247.8, 102.2), turned to -90 degrees
- moved R22 19.4 mm to (260.7, 120.0), turned to 180 degrees
- moved R23 17.7 mm to (260.7, 122.0), turned to 180 degrees
- moved R21 8.82 mm to (261.4, 117.1), turned to -90 degrees
- moved R6 1.53 mm to (260.2, 104.4)
- moved R3 1.51 mm to (261.0, 95.0)
- moved FL2 1.37 mm to (262.0, 104.7)
- moved R20 1.32 mm to (263.4, 110.7)
- moved J4 1.25 mm to (242.6, 93.3)
- moved C10 1.16 mm to (260.6, 109.0)
- moved U1 1.16 mm to (256.4, 114.5)
- moved Y1 1.10 mm to (272.2, 95.9)
- moved C9 0.85 mm to (257.8, 106.7)
- moved C38 0.56 mm to (260.7, 106.9)
- moved J7 0.29 mm to (267.6, 62.9)
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Routing:
- net GND: track 0.83 -> 71.1 mm, vias 0 -> 52
- net +3V3: track 49.0 -> 92.5 mm
- net /USB Hub/RXN: track 2.31 -> 19.3 mm, vias 1 -> 2
- net /USB Hub/RXP: track 2.68 -> 19.3 mm, vias 1 -> 2
- net +5V_WiFi: track 39.4 -> 53.9 mm, vias 17 -> 4
- net /USB Hub/ferrite: track 30.0 -> 39.9 mm, vias 5 -> 4
- net /USB Hub/USB4_N: track 32.7 -> 42.4 mm
- net /USB Hub/USB4_P: track 32.8 -> 42.1 mm
- net /USB Hub/USB1_N: track 34.1 -> 27.0 mm
- net /USB Hub/USB1_P: track 32.3 -> 27.1 mm
- net /USB Hub/TXN: track 17.3 -> 12.8 mm, vias 0 -> 2
- net /USB Hub/USB3_P: track 25.0 -> 28.3 mm
- net Net-(IC1-TXD2/GPIO6/PORT_SWAP): track 0.00 -> 3.21 mm
- net /USBD_UP_P: track 25.3 -> 22.3 mm
- net /USB Hub/USB3_N: track 25.3 -> 28.1 mm
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- added copper zone on F.Cu, net +5V_WiFi
- added copper zone on In1.Cu, net GND
- added copper zone on In2.Cu, net GND
Other:
- copper layers 2 -> 4

Commit message: push after error check
Parts:
- IC1: value LAN9500AI-ABZJ-TR -> QFN50P800X800X100-57N-D
- U1: value BL-M8812EU2 -> Untitled
- moved R22 1.49 mm to (260.7, 118.5)
- moved R20 1.28 mm to (263.3, 109.4)
- moved J5 1.21 mm to (268.5, 126.9)
- moved R24 1.19 mm to (272.1, 108.3)
- moved R25 1.19 mm to (270.1, 108.3)
- moved R23 1.12 mm to (260.7, 120.9)
- moved R21 1.12 mm to (260.7, 116.2), turned to 180 degrees
- moved T1 1.10 mm to (268.0, 116.7)
- moved C6 1.09 mm to (267.9, 107.7)
- moved J3 1.00 mm to (253.4, 126.9)
- moved J4 0.85 mm to (243.5, 93.2)
- moved J7 0.78 mm to (267.8, 63.6)
- moved J6 0.78 mm to (253.2, 63.6)
Routing:
- net +5V_WiFi: track 53.9 -> 11.4 mm, vias 4 -> 5
- net +3V3: track 92.5 -> 82.0 mm, vias 5 -> 3
- net /USB Hub/RX_N: track 23.5 -> 19.9 mm
- net /USB Hub/TX_P: track 32.2 -> 28.6 mm
- net /USB Hub/TX_N: track 32.0 -> 28.9 mm
- net +5V_Radxa: track 147.6 -> 145.4 mm
- net /USB Hub/RX_P: track 23.2 -> 21.1 mm
- net /UART4_RX: track 52.8 -> 51.1 mm
- net /USB Hub/TXN: track 12.8 -> 14.0 mm
- net /USB Hub/USB4_N: track 42.4 -> 41.2 mm
- net /USB Hub/RXP: track 19.3 -> 18.2 mm
- net /USB Hub/RXN: track 19.3 -> 18.4 mm
- net /USB Hub/TXP: track 13.5 -> 14.4 mm
- net /USB Hub/USB3_P: track 28.3 -> 27.4 mm
- net Net-(IC1-TXD2/GPIO6/PORT_SWAP): track 3.21 -> 3.92 mm
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- added copper zone on B.Cu, net +5V_WiFi
